Commit message: reversed the lidar to match neato node

File: src/neato_simulator/model/hokuyo.urdf.xacro (robot description, xacro)
@@ -24,5 +24,5 @@
  <joint name="hokuyo_joint" type="fixed">
    <axis xyz="0 0 1" />
-   <origin xyz="0 0 0.13" rpy="0 0 0"/>
+   <origin xyz="0 0 0.13" rpy="0 0 -3.14159"/>
    <!--<origin xyz="0 -0.035 0.035" rpy="0 0 0"/>-->
 <parent link="base_link"/>
@@ -36,8 +36,8 @@
 	  <scan>
 	    <horizontal>
-	      <samples>360</samples>
+	      <samples>361</samples>
 	      <resolution>1</resolution>
-	      <min_angle>0</min_angle>
-	      <max_angle>6.283185</max_angle>
+	      <min_angle>-3.14159265</min_angle>
+	      <max_angle>3.14159265</max_angle>
 	    </horizontal>
 	  </scan>
